File: PCB/HumidTempSleep_Feather/HumidTempSleep_Feather_001.brd (EAGLE design)
At the start: 100 x 80 mm, 9 parts

Commit message: Added prototype jumpers
Parts:
- added J6, J7, J8: (no value), SparkFun-Connectors:1X10
- moved J1 2.03 mm to (48.5, 63.5)
- moved R1 1.27 mm to (51.1, 54.6)
- moved R2 1.27 mm to (48.3, 54.6)
- moved J4 0.25 mm to (53.8, 53.3)
Connections:
- net 3V: now also J6.10, J6.8, J6.9
- net GND: now also J7.10, J7.8, J7.9
- net USB: now also J8.10, J8.8, J8.9
Routing:
- net GND: track 43.4 -> 56.4 mm, vias 0 -> 1
- net USB: track 2.54 -> 12.2 mm
- net 3V: track 55.1 -> 62.2 mm
- net VBAT: track 13.8 -> 12.6 mm
- net N$24: track 9.26 -> 10.5 mm
- net DATA: track 16.6 -> 15.8 mm
Other:
- board text added: "1"
- board text added: "20191211"
- board text added: "3V"
- board text added: "BLINKERTON LABS"
- board text added: "DHT TEMP+SLEEP"
- board text added: "SLEEP JUMPER"
- board text added: "USB"
- board text added: "VBATT JUMPER"
